File: hardware/seven_segment.kicad_pcb (KiCad board)
At the start: 2 copper layers, 95.2 x 50.8 mm, 50 parts, among them J1 Conn_02x08_Odd_Even, J2 PJ-102AH, J3 7761, J4 7761, J5 Conn_01x02, SW1 SW_Push, SW2 SW_Push, SW3 SW_Push, SW4 SW_Push, U1 STM32F051K8Ux, U10 TPS22810DRV, U11 TPS22810DRV, U12 TPS22810DRV, U13 TPS22810DRV, U2 ULN2003A, U3 ULN2003A, U4 AP1117-33, U5 TPS22810DRV, U6 74HC238, U7 TPS22810DRV, U8 TPS22810DRV, U9 TPS22810DRV

Commit message: hardware: Start work on version 2
Parts:
- removed C4: C, Resistor_SMD:R_0603_1608Metric
- removed DISP1, DISP2, DISP3, DISP4, DISP5, DISP6, DISP7, DISP8: Conn_01x01, klauke:2025
- removed J4: 7761, 7761:KEYSTONE_7761
- removed J5: Conn_01x02, Connector_PinHeader_2.54mm:PinHeader_1x02_P2.54mm_Vertical
- removed R7, R8: R, Resistor_SMD:R_0603_1608Metric
- removed SW4: SW_Push, pushbutton:TO_6083716_WRE
- removed U13: TPS22810DRV, Package_SON:WSON-6-1EP_2x2mm_P0.65mm_EP1x1.6mm
- added BOOT0: BOOT0, TestPoint:TestPoint_Pad_D1.5mm, F.Cu at (117.5, 136.5)
- C1, C2, C3, R1, R2, R3, U4: moved to B.Cu
- J1: value Conn_02x08_Odd_Even -> Conn_01x16
- J3: value 7761 -> Conn_01x04; footprint 7761:KEYSTONE_7761 -> Connector_JST:JST_EH_B4B-EH-A_1x04_P2.50mm_Vertical
- U10, U7, U8, U9: value TPS22810DRV -> TPS22810DBVT; footprint Package_SON:WSON-6-1EP_2x2mm_P0.65mm_EP1x1.6mm -> Package_TO_SOT_SMD:SOT-23-6
- U11: value TPS22810DRV -> STM32F051C8Tx; footprint Package_SON:WSON-6-1EP_2x2mm_P0.65mm_EP1x1.6mm -> Package_QFP:LQFP-48_7x7mm_P0.5mm
- U12: value TPS22810DRV -> STM32F051C8Ux; footprint Package_SON:WSON-6-1EP_2x2mm_P0.65mm_EP1x1.6mm -> Package_DFN_QFN:QFN-48-1EP_7x7mm_P0.5mm_EP5.6x5.6mm
- U5: value TPS22810DRV -> 74HC595; footprint Package_SON:WSON-6-1EP_2x2mm_P0.65mm_EP1x1.6mm -> Package_SO:SOP-16_4.55x10.3mm_P1.27mm; moved to B.Cu
- U6: value 74HC238 -> 74HC595; footprint Package_SO:SOIC-16W_5.3x10.2mm_P1.27mm -> Package_SO:SOP-16_4.55x10.3mm_P1.27mm; moved to B.Cu
- moved U4 67.9 mm to (83.2, 144.1), turned to 0 degrees
- moved J2 67.2 mm to (83.8, 127.6)
- moved J3 58.8 mm to (129.5, 154.0), turned to 180 degrees
- moved C5 58.6 mm to (82.7, 140.3)
- moved C6 58.6 mm to (82.7, 148.6)
- moved U5 56.5 mm to (107.3, 145.4), turned to 90 degrees
- moved UART1 42.4 mm to (121.9, 103.5)
- moved U10 36.2 mm to (114.9, 146.7), turned to -90 degrees
- moved U8 34.9 mm to (122.6, 146.7), turned to -90 degrees
- moved R9 28.2 mm to (114.9, 136.5), turned to 90 degrees
- moved U1 27.5 mm to (118.7, 141.6), turned to -90 degrees
- moved U6 25.6 mm to (95.9, 145.4), turned to 90 degrees
- moved SWD1 23.1 mm to (128.9, 135.3), turned to 0 degrees
- moved C7 22.4 mm to (104.8, 132.1)
- moved C8 22.4 mm to (100.3, 132.1)
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Connections:
- R9 pad 1: Net-(J5-Pad1) -> GND
- R9 pad 2: +3V3 -> Net-(BOOT0-Pad1)
- SWD1 pad 3: /SWDIO -> /SWCLK
- SWD1 pad 4: /SWCLK -> /SWDIO
- U1 pad 10: /setE -> unconnected-(U1-Pad10)
- U1 pad 11: /setF -> /SCK
- U1 pad 12: /setG -> /MISO
- U1 pad 13: /clrA -> /MOSI
- U1 pad 14: /clrB -> unconnected-(U1-Pad14)
- U1 pad 15: /clrC -> unconnected-(U1-Pad15)
- U1 pad 16: /clrD -> unconnected-(U1-Pad16)
- U1 pad 18: /clrE -> Net-(U1-Pad18)
- U1 pad 21: /clrF -> unconnected-(U1-Pad21)
- U1 pad 22: /clrG -> unconnected-(U1-Pad22)
- U1 pad 23: /SWDIO -> unconnected-(U1-Pad23)
- U1 pad 24: /SWCLK -> /SWDIO
- U1 pad 25: /sel_en -> /SWCLK
- U1 pad 26: /sel2 -> unconnected-(U1-Pad26)
- U1 pad 27: /sel1 -> unconnected-(U1-Pad27)
- U1 pad 28: /sel0 -> unconnected-(U1-Pad28)
- U1 pad 31: Net-(J5-Pad1) -> Net-(BOOT0-Pad1)
- U1 pad 32: Net-(R8-Pad1) -> unconnected-(U1-Pad32)
- U1 pad 6: /setA -> Net-(U1-Pad6)
- U1 pad 7: /setB -> Net-(U1-Pad7)
- U1 pad 8: /setC -> Net-(U1-Pad8)
- U1 pad 9: /setD -> Net-(U1-Pad9)
- U10 pad 1: Net-(DISP3-Pad1) -> +12V
- U10 pad 2: unconnected-(U10-Pad2) -> GND
- U10 pad 3: unconnected-(U10-Pad3) -> Net-(U1-Pad9)
- U10 pad 4: GND -> unconnected-(U10-Pad4)
- U10 pad 5: /D3 -> unconnected-(U10-Pad5)
- U10 pad 6: +12V -> Net-(U10-Pad6)
- U11 pad 1: Net-(DISP7-Pad1) -> unconnected-(U11-Pad1)
- U11 pad 4: GND -> unconnected-(U11-Pad4)
- U11 pad 5: /D7 -> unconnected-(U11-Pad5)
- U11 pad 6: +12V -> unconnected-(U11-Pad6)
- U11 pad 7: GND -> unconnected-(U11-Pad7)
- U12 pad 1: Net-(DISP4-Pad1) -> unconnected-(U12-Pad1)
- U12 pad 4: GND -> unconnected-(U12-Pad4)
- U12 pad 5: /D4 -> unconnected-(U12-Pad5)
- U12 pad 6: +12V -> unconnected-(U12-Pad6)
- U12 pad 7: GND -> unconnected-(U12-Pad7)
- U2 pad 1: /setG -> Net-(U2-Pad1)
- U2 pad 10: Net-(J1-Pad14) -> Net-(J1-Pad9)
- U2 pad 11: Net-(J1-Pad10) -> Net-(J1-Pad8)
- U2 pad 12: Net-(J1-Pad6) -> Net-(J1-Pad7)
- U2 pad 13: Net-(J1-Pad4) -> Net-(J1-Pad6)
- U2 pad 14: Net-(J1-Pad7) -> Net-(J1-Pad5)
- U2 pad 15: Net-(J1-Pad11) -> Net-(J1-Pad4)
- U2 pad 16: Net-(J1-Pad13) -> Net-(J1-Pad3)
- U2 pad 2: /setF -> Net-(U2-Pad2)
- U2 pad 3: /setE -> Net-(U2-Pad3)
- U2 pad 4: /setD -> Net-(U2-Pad4)
- U2 pad 5: /setC -> Net-(U2-Pad5)
- U2 pad 6: /setB -> Net-(U2-Pad6)
- U2 pad 7: /setA -> Net-(U2-Pad7)
- U3 pad 1: /clrG -> Net-(U3-Pad1)
- U3 pad 11: Net-(J1-Pad12) -> Net-(J1-Pad15)
- U3 pad 12: Net-(J1-Pad8) -> Net-(J1-Pad14)
- U3 pad 13: Net-(J1-Pad3) -> Net-(J1-Pad13)
- U3 pad 14: Net-(J1-Pad5) -> Net-(J1-Pad12)
- U3 pad 15: Net-(J1-Pad9) -> Net-(J1-Pad11)
- U3 pad 16: Net-(J1-Pad15) -> Net-(J1-Pad10)
- U3 pad 2: /clrF -> Net-(U3-Pad2)
- U3 pad 3: /clrE -> Net-(U3-Pad3)
- U3 pad 4: /clrD -> Net-(U3-Pad4)
- U3 pad 5: /clrC -> Net-(U3-Pad5)
- U3 pad 6: /clrB -> Net-(U3-Pad6)
- U3 pad 7: /clrA -> Net-(U3-Pad7)
- U5 pad 1: Net-(DISP1-Pad1) -> Net-(U2-Pad1)
- U5 pad 2: unconnected-(U5-Pad2) -> Net-(U2-Pad2)
- U5 pad 3: unconnected-(U5-Pad3) -> Net-(U2-Pad3)
- U5 pad 4: GND -> Net-(U2-Pad4)
- U5 pad 5: /D1 -> Net-(U2-Pad5)
- U5 pad 6: +12V -> Net-(U2-Pad6)
- U5 pad 7: GND -> Net-(U2-Pad7)
- U6 pad 1: /sel0 -> Net-(U3-Pad1)
- U6 pad 10: /D6 -> +3V3
- U6 pad 11: /D5 -> /SCK
- U6 pad 12: /D4 -> /SCK
- U6 pad 13: /D3 -> Net-(U1-Pad18)
- U6 pad 14: /D2 -> Net-(U5-Pad9)
- U6 pad 15: /D1 -> unconnected-(U6-Pad15)
- U6 pad 2: /sel1 -> Net-(U3-Pad2)
- U6 pad 3: /sel2 -> Net-(U3-Pad3)
- U6 pad 4: GND -> Net-(U3-Pad4)
- U6 pad 5: GND -> Net-(U3-Pad5)
- U6 pad 6: /sel_en -> Net-(U3-Pad6)
- U6 pad 7: /D8 -> Net-(U3-Pad7)
- U6 pad 9: /D7 -> unconnected-(U6-Pad9)
- U7 pad 1: Net-(DISP5-Pad1) -> +12V
- U7 pad 2: unconnected-(U7-Pad2) -> GND
- U7 pad 3: unconnected-(U7-Pad3) -> Net-(U1-Pad6)
- U7 pad 4: GND -> unconnected-(U7-Pad4)
- U7 pad 5: /D5 -> unconnected-(U7-Pad5)
- U7 pad 6: +12V -> Net-(U7-Pad6)
- U8 pad 1: Net-(DISP2-Pad1) -> +12V
- U8 pad 2: unconnected-(U8-Pad2) -> GND
- U8 pad 3: unconnected-(U8-Pad3) -> Net-(U1-Pad7)
- U8 pad 4: GND -> unconnected-(U8-Pad4)
- U8 pad 5: /D2 -> unconnected-(U8-Pad5)
- U8 pad 6: +12V -> Net-(U8-Pad6)
- U9 pad 1: Net-(DISP6-Pad1) -> +12V
- U9 pad 2: unconnected-(U9-Pad2) -> GND
- U9 pad 3: unconnected-(U9-Pad3) -> Net-(U1-Pad8)
- U9 pad 4: GND -> unconnected-(U9-Pad4)
- U9 pad 5: /D6 -> unconnected-(U9-Pad5)
- U9 pad 6: +12V -> Net-(U9-Pad6)
Routing:
- net +3V3: track 151.6 -> 1.34 mm, vias 4 -> 0
- net +12V: track 130.8 -> 29.2 mm, vias 14 -> 0
- net GND: track 84.9 -> 13.0 mm, vias 83 -> 2
- net /D1: track 45.5 -> 0.00 mm
- net Net-(R8-Pad1): track 45.3 -> 0.00 mm, vias 2 -> 0
- net /D2: track 40.5 -> 0.00 mm
- net Net-(J1-Pad15): track 44.0 -> 4.41 mm
- net /sel0: track 37.3 -> 0.00 mm
- net Net-(R6-Pad1): track 36.1 -> 0.00 mm, vias 2 -> 0
- net Net-(J1-Pad16): track 43.5 -> 7.48 mm
- net /D3: track 35.4 -> 0.00 mm
- net /sel1: track 34.6 -> 0.00 mm
- net /sel2: track 31.8 -> 0.00 mm
- net /D4: track 30.6 -> 0.00 mm
- net Net-(J1-Pad13): track 31.5 -> 4.41 mm
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- removed copper zone on F.Cu, net +12V
- removed copper zone on F.Cu, net +3V3
- removed copper zone on B.Cu, net GND
- removed copper zone on F.Cu, net GND

Commit message: hardware: Version 2
Parts:
- removed C3: C, Resistor_SMD:R_0603_1608Metric
- removed SW1, SW3: SW_Push, pushbutton:TO_6083716_WRE
- removed U12: STM32F051C8Ux, Package_DFN_QFN:QFN-48-1EP_7x7mm_P0.5mm_EP5.6x5.6mm
- added BT1: Battery_Cell, Battery:BatteryHolder_Keystone_3000_1x12mm, B.Cu at (167.0, 119.4)
- added C10: C, Resistor_SMD:R_0402_1005Metric_Pad0.72x0.64mm_HandSolder, F.Cu at (170.8, 116.2)
- added C4: C, Resistor_SMD:R_0402_1005Metric_Pad0.72x0.64mm_HandSolder, F.Cu at (170.8, 113.7)
- added D1: LED, Connector_PinHeader_2.54mm:PinHeader_1x02_P2.54mm_Vertical, F.Cu at (121.9, 104.1)
- added R7: 10k, Resistor_SMD:R_0603_1608Metric, F.Cu at (125.7, 102.9)
- added RST1: SW_Push, pushbutton:TO_6083716_WRE, F.Cu at (166.1, 105.4)
- added Y1: Crystal, Crystal:Crystal_SMD_3215-2Pin_3.2x1.5mm, F.Cu at (169.0, 114.9)
- C5, C6: footprint Capacitor_THT:CP_Radial_D7.5mm_P2.50mm -> Capacitor_SMD:CP_Elec_6.3x5.9
- C7, C8, C9: moved to B.Cu
- R3: value R -> 10k; moved to F.Cu
- R6: value R -> 10k
- R9: value R -> 10k; moved to B.Cu
- U11: value STM32F051C8Tx -> MCP7940N-xSN; footprint Package_QFP:LQFP-48_7x7mm_P0.5mm -> Package_SO:SO-8_3.9x4.9mm_P1.27mm
- moved C1 73.0 mm to (162.6, 104.8)
- moved R1 73.0 mm to (162.6, 106.7)
- moved R4 73.0 mm to (162.6, 106.7), turned to 0 degrees
- moved C8 59.0 mm to (157.5, 117.5), turned to -90 degrees
- moved C9 58.0 mm to (155.6, 108.6)
- moved R9 52.2 mm to (158.6, 108.0), turned to 0 degrees
- moved J1 52.1 mm to (147.9, 115.6)
- moved C7 51.0 mm to (153.7, 117.5), turned to -90 degrees
- moved C2 50.7 mm to (152.4, 104.8)
- moved U2 50.4 mm to (141.0, 107.9)
- moved U5 50.4 mm to (141.0, 107.9)
- moved U3 50.4 mm to (129.5, 107.9)
- moved U6 50.4 mm to (129.5, 107.9)
- moved C6 50.2 mm to (107.5, 105.0), turned to 180 degrees
- moved BOOT0 50.0 mm to (159.4, 109.2)
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Connections:
- R3 pad 1: Net-(C3-Pad1) -> /SDA
- R6 pad 1: Net-(R6-Pad1) -> /SCL
- R6 pad 2: Net-(C3-Pad1) -> +3V3
- U1 pad 10: unconnected-(U1-Pad10) -> Net-(U1-Pad10)
- U1 pad 14: unconnected-(U1-Pad14) -> Net-(U1-Pad14)
- U1 pad 15: unconnected-(U1-Pad15) -> Net-(U1-Pad15)
- U1 pad 16: unconnected-(U1-Pad16) -> Net-(U1-Pad16)
- U1 pad 28: unconnected-(U1-Pad28) -> Net-(U1-Pad28)
- U1 pad 29: Net-(R5-Pad1) -> /SCL
- U1 pad 30: Net-(R6-Pad1) -> /SDA
- U1 pad 6: Net-(U1-Pad6) -> unconnected-(U1-Pad6)
- U1 pad 7: Net-(U1-Pad7) -> unconnected-(U1-Pad7)
- U1 pad 8: Net-(U1-Pad8) -> Net-(R5-Pad1)
- U10 pad 3: Net-(U1-Pad9) -> Net-(U1-Pad18)
- U11 pad 1: unconnected-(U11-Pad1) -> Net-(C10-Pad1)
- U11 pad 2: unconnected-(U11-Pad2) -> Net-(C4-Pad1)
- U11 pad 3: unconnected-(U11-Pad3) -> Net-(BT1-Pad1)
- U11 pad 4: unconnected-(U11-Pad4) -> GND
- U11 pad 5: unconnected-(U11-Pad5) -> /SDA
- U11 pad 6: unconnected-(U11-Pad6) -> /SCL
- U11 pad 7: unconnected-(U11-Pad7) -> Net-(U1-Pad28)
- U11 pad 8: unconnected-(U11-Pad8) -> +3V3
- U5 pad 13: Net-(U1-Pad18) -> Net-(U1-Pad10)
- U6 pad 13: Net-(U1-Pad18) -> Net-(U1-Pad10)
- U7 pad 3: Net-(U1-Pad6) -> Net-(U1-Pad14)
- U8 pad 3: Net-(U1-Pad7) -> Net-(U1-Pad15)
- U9 pad 3: Net-(U1-Pad8) -> Net-(U1-Pad16)
Routing:
- net +3V3: track 1.34 -> 117.9 mm, vias 0 -> 6
- net Net-(U1-Pad14): track 0.00 -> 45.9 mm, vias 0 -> 2
- net Net-(U1-Pad16): track 0.00 -> 41.2 mm
- net Net-(U1-Pad15): track 0.00 -> 34.3 mm
- net Net-(U1-Pad9): track 0.00 -> 33.7 mm
- net +12V: track 29.2 -> 62.6 mm, vias 0 -> 4
- net Net-(U1-Pad10): track 0.00 -> 33.2 mm, vias 0 -> 1
- net Net-(U1-Pad18): track 15.6 -> 45.7 mm
- net /SWCLK: track 0.00 -> 22.3 mm
- net /SWDIO: track 0.00 -> 21.4 mm
- net GND: track 13.0 -> 31.0 mm, vias 2 -> 93
- net /MOSI: track 0.00 -> 18.0 mm, vias 0 -> 1
- net /UART_RX: track 0.00 -> 14.6 mm
- net /SCK: track 22.6 -> 36.0 mm, vias 0 -> 2
- net /UART_TX: track 0.00 -> 13.1 mm
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- added copper zone on B.Cu, net +3V3
- added copper zone on B.Cu, net GND
- added copper zone on F.Cu, net GND
Other:
- board size 95.2 x 50.8 mm -> 74 x 34 mm
- board text added: "Hammond 1551KBK max.height 10.4mm"

Commit message: hardware: revision 3
Parts:
- removed BOOT0: BOOT0, TestPoint:TestPoint_Pad_D1.5mm
- removed BT1: Battery_Cell, Battery:BatteryHolder_Keystone_3000_1x12mm
- removed C10: C, Resistor_SMD:R_0402_1005Metric_Pad0.72x0.64mm_HandSolder
- removed C5, C6: C_Polarized, Capacitor_SMD:CP_Elec_6.3x5.9
- removed D1: LED, Connector_PinHeader_2.54mm:PinHeader_1x02_P2.54mm_Vertical
- removed SWD1, UART1: Conn_01x04, Connector_PinHeader_2.54mm:PinHeader_1x04_P2.54mm_Vertical
- removed U10, U8, U9: TPS22810DBVT, Package_TO_SOT_SMD:SOT-23-6
- removed U11: MCP7940N-xSN, Package_SO:SO-8_3.9x4.9mm_P1.27mm
- removed Y1: Crystal, Crystal:Crystal_SMD_3215-2Pin_3.2x1.5mm
- added C3: 10p, Resistor_SMD:R_0603_1608Metric, F.Cu at (151.1, 108.6)
- added J5: Conn_01x06, Connector:Tag-Connect_TC2030-IDC-NL_2x03_P1.27mm_Vertical, F.Cu at (144.8, 104.1)
- added K1: ~, 00_customfootprints:G6DN-1A-SL, B.Cu at (111.1, 113.2)
- added K2: ~, 00_customfootprints:G6DN-1A-SL, F.Cu at (111.1, 113.2)
- added K3: ~, 00_customfootprints:G6DN-1A-SL, B.Cu at (131.4, 113.2)
- added K4: ~, 00_customfootprints:G6DN-1A-SL, F.Cu at (131.4, 113.2)
- added L1: 2.2u, Inductor_SMD:L_Vishay_IHLP-1212, F.Cu at (146.7, 112.0)
- added R10: 10k, Resistor_SMD:R_0603_1608Metric, B.Cu at (144.9, 112.0)
- added R11: 10k, Resistor_SMD:R_0603_1608Metric, F.Cu at (144.1, 116.3)
- added R8: R, Resistor_SMD:R_0603_1608Metric, F.Cu at (127.6, 114.9)
- C4: value C -> 0.1u; footprint Resistor_SMD:R_0402_1005Metric_Pad0.72x0.64mm_HandSolder -> Resistor_SMD:R_0603_1608Metric
- C7, C8: value C -> 22u; footprint Resistor_SMD:R_0805_2012Metric -> Capacitor_SMD:C_0805_2012Metric; moved to F.Cu
- C9: value C -> 10u; footprint Resistor_SMD:R_0805_2012Metric -> Capacitor_SMD:C_0805_2012Metric; moved to F.Cu
- J1: footprint Connector_PinHeader_2.54mm:PinHeader_2x08_P2.54mm_Horizontal -> Connector_PinHeader_2.54mm:PinHeader_2x08_P2.54mm_Vertical
- R1, R2: value R -> 10k; moved to F.Cu
- R3, R7: value 10k -> R; moved to B.Cu
- R4, R5: moved to B.Cu
- R6: value 10k -> R
- R9: value 10k -> 33.2k
- U1: value STM32F051K8Ux -> ESP32-WROOM-32E; footprint Package_DFN_QFN:QFN-32-1EP_5x5mm_P0.5mm_EP3.45x3.45mm -> RF_Module:ESP32-WROOM-32D
- U2, U3: footprint Package_SO:SOP-16_4.55x10.3mm_P1.27mm -> Package_SO:SOP-16_3.9x9.9mm_P1.27mm; moved to B.Cu
- U4: value AP1117-33 -> TPS562200; footprint Package_TO_SOT_SMD:SOT-223-3_TabPin2 -> Package_TO_SOT_SMD:SOT-23-6; moved to F.Cu
- U5, U6: footprint Package_SO:SOP-16_4.55x10.3mm_P1.27mm -> Package_SO:SOP-16_3.9x9.9mm_P1.27mm
- U7: value TPS22810DBVT -> ULN2003A; footprint Package_TO_SOT_SMD:SOT-23-6 -> Package_SO:SOP-16_3.9x9.9mm_P1.27mm
- moved R6 54.5 mm to (107.5, 114.9), turned to 0 degrees
- moved R3 49.0 mm to (114.9, 115.6), turned to 180 degrees
- moved U6 38.9 mm to (168.3, 111.8), turned to 0 degrees
- moved U4 38.6 mm to (146.7, 116.5), turned to -90 degrees
- moved U5 31.0 mm to (168.3, 122.6), turned to 0 degrees
- moved U3 30.7 mm to (160.0, 111.8), turned to 180 degrees
- moved U2 24.0 mm to (160.0, 122.6), turned to 180 degrees
- moved C4 21.8 mm to (149.2, 116.6)
- moved J3 17.4 mm to (114.6, 130.9), turned to 90 degrees
- moved R7 15.9 mm to (135.3, 115.6)
- moved C9 12.6 mm to (143.8, 113.0)
- moved R9 12.6 mm to (146.7, 112.0), turned to -90 degrees
- moved U7 10.9 mm to (122.6, 122.6), turned to 90 degrees
- moved R1 10.8 mm to (153.0, 111.8), turned to -90 degrees
- moved U1 10.3 mm to (164.0, 118.0), turned to 180 degrees
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Connections:
- C1 pad 1: Net-(C1-Pad1) -> Net-(U1-IO19)
- C2 pad 1: Net-(C2-Pad1) -> Net-(U1-IO4)
- C4 pad 1: Net-(C4-Pad1) -> Net-(U4-VBST)
- C4 pad 2: GND -> Net-(U4-SW)
- C9 pad 1: +3V3 -> +12V
- J1 pad 10: Net-(J1-Pad10) -> Net-(J1-Pin_10)
- J1 pad 11: Net-(J1-Pad11) -> Net-(J1-Pin_11)
- J1 pad 12: Net-(J1-Pad12) -> Net-(J1-Pin_12)
- J1 pad 14: Net-(J1-Pad14) -> Net-(J1-Pin_14)
- J1 pad 15: Net-(J1-Pad15) -> Net-(J1-Pin_15)
- J1 pad 16: Net-(J1-Pad16) -> Net-(J1-Pin_16)
- J1 pad 3: Net-(J1-Pad3) -> Net-(J1-Pin_3)
- J1 pad 4: Net-(J1-Pad4) -> Net-(J1-Pin_4)
- J1 pad 5: Net-(J1-Pad5) -> Net-(J1-Pin_5)
- J1 pad 7: Net-(J1-Pad7) -> Net-(J1-Pin_7)
- J1 pad 8: Net-(J1-Pad8) -> Net-(J1-Pin_8)
- J1 pad 9: Net-(J1-Pad9) -> Net-(J1-Pin_9)
- J3 pad 1: Net-(J3-Pad1) -> Net-(J3-Pin_1)
- R1 pad 1: Net-(C1-Pad1) -> +3V3
- R1 pad 2: +3V3 -> Net-(U1-IO16)
- R2 pad 1: Net-(C2-Pad1) -> +3V3
- R2 pad 2: +3V3 -> Net-(J5-Pin_1)
- R3 pad 1: /SDA -> Net-(K1-Pad2)
- R3 pad 2: +3V3 -> +12V
- R4 pad 1: Net-(R4-Pad1) -> Net-(U1-IO19)
- R4 pad 2: Net-(C1-Pad1) -> Net-(R4-Pad2)
- R5 pad 1: Net-(R5-Pad1) -> Net-(U1-IO4)
- R5 pad 2: Net-(C2-Pad1) -> Net-(R5-Pad2)
- R6 pad 1: /SCL -> Net-(K2-Pad2)
- R6 pad 2: +3V3 -> +12V
- R7 pad 1: Net-(U1-Pad9) -> Net-(K3-Pad2)
- R7 pad 2: Net-(D1-Pad1) -> +12V
- R9 pad 1: GND -> +3V3
- R9 pad 2: Net-(BOOT0-Pad1) -> Net-(U4-VFB)
- RST1 pad 1: Net-(C1-Pad1) -> Net-(R4-Pad2)
- SW2 pad 1: Net-(C2-Pad1) -> Net-(R5-Pad2)
- U1 pad 1: +3V3 -> GND
- U1 pad 10: Net-(U1-Pad10) -> Net-(U1-IO25)
- U1 pad 11: /SCK -> unconnected-(U1-IO26-Pad11)
- U1 pad 12: /MISO -> unconnected-(U1-IO27-Pad12)
- U1 pad 13: /MOSI -> unconnected-(U1-IO14-Pad13)
- U1 pad 14: Net-(U1-Pad14) -> unconnected-(U1-IO12-Pad14)
- U1 pad 15: Net-(U1-Pad15) -> GND
- U1 pad 16: Net-(U1-Pad16) -> unconnected-(U1-IO13-Pad16)
- U1 pad 17: +3V3 -> unconnected-(U1-NC-Pad17)
- U1 pad 18: Net-(U1-Pad18) -> unconnected-(U1-NC-Pad18)
- U1 pad 19: /UART_TX -> unconnected-(U1-NC-Pad19)
- U1 pad 2: unconnected-(U1-Pad2) -> +3V3
- U1 pad 20: /UART_RX -> unconnected-(U1-NC-Pad20)
- U1 pad 24: /SWDIO -> unconnected-(U1-IO2-Pad24)
- U1 pad 25: /SWCLK -> Net-(J5-Pin_6)
- U1 pad 26: unconnected-(U1-Pad26) -> Net-(U1-IO4)
- U1 pad 27: unconnected-(U1-Pad27) -> Net-(U1-IO16)
- U1 pad 28: Net-(U1-Pad28) -> Net-(U1-IO17)
- U1 pad 29: /SCL -> unconnected-(U1-IO5-Pad29)
- U1 pad 3: unconnected-(U1-Pad3) -> Net-(J5-Pin_1)
- U1 pad 30: /SDA -> Net-(U1-IO18)
- U1 pad 31: Net-(BOOT0-Pad1) -> Net-(U1-IO19)
- U1 pad 33: GND -> unconnected-(U1-IO21-Pad33)
- U1 pad 4: Net-(R4-Pad1) -> unconnected-(U1-SENSOR_VP-Pad4)
- U1 pad 5: +3V3 -> unconnected-(U1-SENSOR_VN-Pad5)
- U1 pad 8: Net-(R5-Pad1) -> Net-(U1-IO32)
- U1 pad 9: Net-(U1-Pad9) -> Net-(U1-IO33)
- U2 pad 1: Net-(U2-Pad1) -> Net-(U2-I1)
- U2 pad 10: Net-(J1-Pad9) -> Net-(J1-Pin_3)
- U2 pad 11: Net-(J1-Pad8) -> Net-(J1-Pin_4)
- U2 pad 12: Net-(J1-Pad7) -> Net-(J1-Pin_5)
- U2 pad 14: Net-(J1-Pad5) -> Net-(J1-Pin_7)
- U2 pad 15: Net-(J1-Pad4) -> Net-(J1-Pin_8)
- U2 pad 16: Net-(J1-Pad3) -> Net-(J1-Pin_9)
- U2 pad 2: Net-(U2-Pad2) -> Net-(U2-I2)
- U2 pad 3: Net-(U2-Pad3) -> Net-(U2-I3)
- U2 pad 5: Net-(U2-Pad5) -> Net-(U2-I5)
- U2 pad 6: Net-(U2-Pad6) -> Net-(U2-I6)
- U2 pad 7: Net-(U2-Pad7) -> Net-(U2-I7)
- U3 pad 1: Net-(U3-Pad1) -> Net-(U3-I1)
- U3 pad 10: Net-(J1-Pad16) -> Net-(J1-Pin_10)
- U3 pad 11: Net-(J1-Pad15) -> Net-(J1-Pin_11)
- U3 pad 12: Net-(J1-Pad14) -> Net-(J1-Pin_12)
- U3 pad 14: Net-(J1-Pad12) -> Net-(J1-Pin_14)
- U3 pad 15: Net-(J1-Pad11) -> Net-(J1-Pin_15)
- U3 pad 16: Net-(J1-Pad10) -> Net-(J1-Pin_16)
- U3 pad 2: Net-(U3-Pad2) -> Net-(U3-I2)
- U3 pad 3: Net-(U3-Pad3) -> Net-(U3-I3)
- U3 pad 5: Net-(U3-Pad5) -> Net-(U3-I5)
- U3 pad 6: Net-(U3-Pad6) -> Net-(U3-I6)
- U3 pad 7: Net-(U3-Pad7) -> Net-(U3-I7)
- U4 pad 2: +3V3 -> Net-(U4-SW)
- U5 pad 1: Net-(U2-Pad1) -> Net-(U2-I7)
- U5 pad 11: /SCK -> Net-(U1-IO25)
- U5 pad 12: /SCK -> Net-(U1-IO25)
- U5 pad 13: Net-(U1-Pad10) -> Net-(U1-IO33)
- U5 pad 14: /MOSI -> Net-(U1-IO32)
- U5 pad 2: Net-(U2-Pad2) -> Net-(U2-I6)
- U5 pad 3: Net-(U2-Pad3) -> Net-(U2-I5)
- U5 pad 5: Net-(U2-Pad5) -> Net-(U2-I3)
- U5 pad 6: Net-(U2-Pad6) -> Net-(U2-I2)
- U5 pad 7: Net-(U2-Pad7) -> Net-(U2-I1)
- U6 pad 1: Net-(U3-Pad1) -> Net-(U3-I7)
- U6 pad 11: /SCK -> Net-(U1-IO25)
- U6 pad 12: /SCK -> Net-(U1-IO25)
- U6 pad 13: Net-(U1-Pad10) -> Net-(U1-IO33)
- U6 pad 2: Net-(U3-Pad2) -> Net-(U3-I6)
- U6 pad 3: Net-(U3-Pad3) -> Net-(U3-I5)
- U6 pad 5: Net-(U3-Pad5) -> Net-(U3-I3)
- U6 pad 6: Net-(U3-Pad6) -> Net-(U3-I2)
- U6 pad 7: Net-(U3-Pad7) -> Net-(U3-I1)
- U7 pad 1: +12V -> Net-(U1-IO17)
- U7 pad 2: GND -> Net-(U1-IO18)
- U7 pad 3: Net-(U1-Pad14) -> Net-(U1-IO22)
- U7 pad 4: unconnected-(U7-Pad4) -> Net-(U1-IO23)
- U7 pad 5: unconnected-(U7-Pad5) -> GND
- U7 pad 6: Net-(J3-Pad1) -> GND
Routing:
- net +3V3: track 117.9 -> 29.3 mm, vias 6 -> 7
- net Net-(J5-Pin_5): track 0.00 -> 47.0 mm, vias 0 -> 2
- net Net-(U1-Pad14): track 45.9 -> 0.00 mm, vias 2 -> 0
- net Net-(U1-Pad18): track 45.7 -> 0.00 mm
- net Net-(U1-IO17): track 0.00 -> 44.5 mm
- net Net-(J5-Pin_3): track 0.00 -> 43.1 mm, vias 0 -> 2
- net Net-(J5-Pin_1): track 0.00 -> 43.0 mm
- net Net-(U1-IO18): track 0.00 -> 42.3 mm
- net Net-(U1-Pad16): track 41.2 -> 0.00 mm
- net Net-(U1-IO22): track 0.00 -> 38.7 mm
- net Net-(U1-IO23): track 0.00 -> 38.4 mm, vias 0 -> 2
- net Net-(J1-Pin_16): track 0.00 -> 36.7 mm
- net /SCK: track 36.0 -> 0.00 mm, vias 2 -> 0
- net Net-(U1-Pad15): track 34.3 -> 0.00 mm
- net +12V: track 62.6 -> 28.4 mm, vias 4 -> 7
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- added copper zone on In2.Cu, net +12V
- added copper zone on In2.Cu, net +3V3
- added copper zone on In1.Cu, net GND
- added copper zone on In2.Cu, net GND
- removed copper zone on B.Cu, net +3V3
Other:
- outline, holes or cut-outs redrawn
- copper layers 2 -> 4

Commit message: hardware: migrate to kicad 8
Connections:
- net Net-(J5-Pin_1) renamed /EN
- net Net-(J5-Pin_3) renamed /RXD0
- net Net-(J5-Pin_5) renamed /TXD0
- net Net-(J5-Pin_6) renamed /IO0

Commit message: hardware: Add net labels to SPI channel
Connections:
- net Net-(U1-IO25) renamed /sreg_sclk
- net Net-(U1-IO32) renamed /sreg_data
- net Net-(U1-IO33) renamed /sreg_oe
Changed lines of the file:
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@@
 	(net 51 "unconnected-(U1-IO5-Pad29)")
 	(net 52 "unconnected-(U1-NC-Pad32)")
-	(net 53 "Net-(U1-IO32)")
+	(net 53 "/sreg_oe")
 	(net 54 "unconnected-(U1-IO26-Pad11)")
 	(net 55 "unconnected-(U1-IO27-Pad12)")
-	(net 56 "Net-(U1-IO25)")
-	(net 57 "Net-(U1-IO33)")
+	(net 56 "/sreg_sclk")
+	(net 57 "/sreg_data")
 	(net 58 "Net-(J3-Pin_1)")
 	(net 59 "Net-(J3-Pin_2)")
@@
 			(size 1.5 0.9)
 			(layers "F.Cu" "F.Paste" "F.Mask")
-			(net 53 "Net-(U1-IO32)")
+			(net 57 "/sreg_data")
 			(pinfunction "IO32")
 			(pintype "bidirectional")
@@
 			(size 1.5 0.9)
 			(layers "F.Cu" "F.Paste" "F.Mask")
-			(net 57 "Net-(U1-IO33)")
+			(net 53 "/sreg_oe")
 			(pinfunction "IO33")
 			(pintype "bidirectional")
@@
 			(size 1.5 0.9)
 			(layers "F.Cu" "F.Paste" "F.Mask")
-			(net 56 "Net-(U1-IO25)")
+			(net 56 "/sreg_sclk")
 			(pinfunction "IO25")
 			(pintype "bidirectional")
@@
 			(layers "B.Cu" "B.Paste" "B.Mask")
 			(roundrect_rratio 0.25)
-			(net 56 "Net-(U1-IO25)")
+			(net 56 "/sreg_sclk")
 			(pinfunction "SRCLK")
 			(pintype "input")
@@
 			(layers "B.Cu" "B.Paste" "B.Mask")
 			(roundrect_rratio 0.25)
-			(net 56 "Net-(U1-IO25)")
+			(net 56 "/sreg_sclk")
 			(pinfunction "RCLK")
 			(pintype "input")
@@
 			(layers "B.Cu" "B.Paste" "B.Mask")
 			(roundrect_rratio 0.25)
-			(net 57 "Net-(U1-IO33)")
+			(net 53 "/sreg_oe")
 			(pinfunction "~{OE}")
 			(pintype "input")
@@
 			(layers "B.Cu" "B.Paste" "B.Mask")
 			(roundrect_rratio 0.25)
-			(net 56 "Net-(U1-IO25)")
+			(net 56 "/sreg_sclk")
 			(pinfunction "SRCLK")
 			(pintype "input")
@@
 			(layers "B.Cu" "B.Paste" "B.Mask")
 			(roundrect_rratio 0.25)
-			(net 56 "Net-(U1-IO25)")
+			(net 56 "/sreg_sclk")
 			(pinfunction "RCLK")
 			(pintype "input")
@@
 			(layers "B.Cu" "B.Paste" "B.Mask")
 			(roundrect_rratio 0.25)
-			(net 57 "Net-(U1-IO33)")
+			(net 53 "/sreg_oe")
 			(pinfunction "~{OE}")
 			(pintype "input")
@@
 			(layers "B.Cu" "B.Paste" "B.Mask")
 			(roundrect_rratio 0.25)
-			(net 53 "Net-(U1-IO32)")
+			(net 57 "/sreg_data")
 			(pinfunction "SER")
 			(pintype "input")
@@
 		(net 34)
 	)
-	(segment
-		(start 169 122.555)
-		(end 171.45 120.105)
-		(width 0.25)
-		(layer "F.Cu")
+	(via
+		(at 172.72 116.205)
+		(size 0.8)
+		(drill 0.4)
+		(layers "F.Cu" "B.Cu")
 		(net 53)
 	)
 	(segment
-		(start 171.45 120.105)
-		(end 171.45 117.66)
+		(start 170.775 112.395)
+		(end 171.929999 112.395)
 		(width 0.25)
-		(layer "F.Cu")
+		(layer "B.Cu")
 		(net 53)
 	)
 	(segment
-		(start 171.45 117.66)
-		(end 171.75 117.36)
+		(start 172.72 113.665)
+		(end 172.72 116.205)
 		(width 0.25)
-		(layer "F.Cu")
+		(layer "B.Cu")
 		(net 53)
 	)
 	(segment
-		(start 171.75 117.36)
-		(end 172.75 117.36)
+		(start 172.72 116.205)
+		(end 172.72 122.555)
 		(width 0.25)
-		(layer "F.Cu")
+		(layer "B.Cu")
 		(net 53)
 	)
-	(via
-		(at 169 122.555)
-		(size 0.8)
-		(drill 0.4)
-		(layers "F.Cu" "B.Cu")
+	(segment
+		(start 172.72 122.555)
+		(end 172.085 123.19)
+		(width 0.25)
+		(layer "B.Cu")
 		(net 53)
 	)
 	(segment
-		(start 169 123.090908)
-		(end 170.369092 124.46)
+		(start 172.085 123.19)
+		(end 170.775 123.19)
 		(width 0.25)
 		(layer "B.Cu")
@@
 	)
 	(segment
-		(start 170.369092 124.46)
-		(end 170.775 124.46)
+		(start 171.929999 112.395)
+		(end 172.72 113.185001)
 		(width 0.25)
 		(layer "B.Cu")
@@
 	)
 	(segment
-		(start 169 122.555)
-		(end 169 123.090908)
+		(start 172.72 113.185001)
+		(end 172.72 113.665)
 		(width 0.25)
 		(layer "B.Cu")
@@
 		(net 56)
 	)
-	(via
-		(at 172.72 116.205)
-		(size 0.8)
-		(drill 0.4)
-		(layers "F.Cu" "B.Cu")
-		(net 57)
-	)
 	(segment
-		(start 170.775 112.395)
-		(end 171.929999 112.395)
+		(start 169 122.555)
+		(end 171.45 120.105)
 		(width 0.25)
-		(layer "B.Cu")
+		(layer "F.Cu")
 		(net 57)
 	)
 	(segment
-		(start 172.72 113.665)
-		(end 172.72 116.205)
+		(start 171.45 120.105)
+		(end 171.45 117.66)
 		(width 0.25)
-		(layer "B.Cu")
+		(layer "F.Cu")
 		(net 57)
 	)
 	(segment
-		(start 172.72 116.205)
-		(end 172.72 122.555)
+		(start 171.45 117.66)
+		(end 171.75 117.36)
 		(width 0.25)
-		(layer "B.Cu")
+		(layer "F.Cu")
 		(net 57)
 	)
 	(segment
-		(start 172.72 122.555)
-		(end 172.085 123.19)
+		(start 171.75 117.36)
+		(end 172.75 117.36)
 		(width 0.25)
-		(layer "B.Cu")
+		(layer "F.Cu")
+		(net 57)
+	)
+	(via
+		(at 169 122.555)
+		(size 0.8)
+		(drill 0.4)
+		(layers "F.Cu" "B.Cu")
 		(net 57)
 	)
 	(segment
-		(start 172.085 123.19)
-		(end 170.775 123.19)
+		(start 169 123.090908)
+		(end 170.369092 124.46)
 		(width 0.25)
 		(layer "B.Cu")
@@
 	)
 	(segment
-		(start 171.929999 112.395)
-		(end 172.72 113.185001)
+		(start 170.369092 124.46)
+		(end 170.775 124.46)
 		(width 0.25)
 		(layer "B.Cu")
@@
 	)
 	(segment
-		(start 172.72 113.185001)
-		(end 172.72 113.665)
+		(start 169 122.555)
+		(end 169 123.090908)
 		(width 0.25)
 		(layer "B.Cu")

Commit message: hardware: Add net labels to segment control pins
Connections:
- net Net-(J1-Pin_10) renamed /set_b
- net Net-(J1-Pin_11) renamed /set_f
- net Net-(J1-Pin_12) renamed /clr_b
- net Net-(J1-Pin_13) renamed /set_g
- net Net-(J1-Pin_14) renamed /set_a
- net Net-(J1-Pin_15) renamed /clr_g
- net Net-(J1-Pin_16) renamed /clr_a
- net Net-(J1-Pin_3) renamed /clr_d
- net Net-(J1-Pin_4) renamed /set_d
- net Net-(J1-Pin_5) renamed /clr_e
- net Net-(J1-Pin_6) renamed /set_c
- net Net-(J1-Pin_7) renamed /set_e
- net Net-(J1-Pin_8) renamed /clr_c
- net Net-(J1-Pin_9) renamed /clr_f
